File: Breakout Adapter v1.0 - LM1117 - AndersV209/ESP12E Breakout Adapter.sch (EAGLE design)
At the start: 10 parts, among them IC1 LM1117-3.3

Commit message: gerberfiles and clean up
Other:
- note added: "ESP8266 Breakout Adapter - ESP-12E custom Date: 21. October 2015 Version: 1.0 License: CC-BY https://creativecommons.org/licenses/by/4.0/"
- note removed: "ESP8266 Breakout Adapter - ESP-07/ESP-12(E) custom Date: 21. October 2015 Version: 0.1 License: CC-BY https://creativecommons.org/licenses/by/4.0/"
Changed lines of the file:
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@@
 <text x="40.64" y="132.08" size="1.778" layer="91">VIN</text>
 <text x="137.16" y="132.08" size="1.778" layer="91">VOUT</text>
-<text x="144.78" y="2.54" size="1.778" layer="91">ESP8266 Breakout Adapter - ESP-07/ESP-12(E) custom
+<text x="144.78" y="2.54" size="1.778" layer="91">ESP8266 Breakout Adapter - ESP-12E custom
 Date: 21. October 2015
-Version: 0.1
+Version: 1.0
 License: CC-BY
 https://creativecommons.org/licenses/by/4.0/</text>
